Commit message: Added Lidar and IMU sensors

File: urdf/construction_robot.urdf (robot description, URDF)
Before this commit: robot construction_robot, 5 links, 4 joints
Links:
- added link imu_link, mass 0.01; collision box size=0.05 0.05 0.02; visual box size=0.05 0.05 0.02
- added link lidar_link, mass 0.2; collision cylinder length=0.08 radius=0.05; visual cylinder length=0.08 radius=0.05
Joints:
- added joint imu_joint: type fixed, parent base_link, child imu_link, origin xyz=0 0 0.15 rpy=0 0 0
- added joint lidar_joint: type fixed, parent base_link, child lidar_link, origin xyz=0 0 0.25 rpy=0 0 0

Commit message: Phase 4 Complete: SLAM Mapping + Web Bridge

File: urdf/construction_robot.urdf (robot description, URDF)
Before this commit: robot construction_robot, 7 links, 6 joints
Joints:
- joint left_wheel_joint: origin xyz=0 0.225 0.1 rpy=-1.5708 0 0 -> xyz=0 0.225 0.1 rpy=1.5708 0 0
